File: Pcb_Diver_Flasher/LED_Flasher/LED_Flasher.kicad_sch (KiCad schematic)
At the start: 30 parts, among them IC101 PIC16LF15313, J101 SKEDD6, SW101 MK15-C2, T101 BUK7880-55A

Commit message: Old PC (v1) removed Latest changes for current schematic routed. Almost ready DRC outstanding.
Parts:
- removed C101: 47µF/10V, Capacitor_SMD:CP_Elec_6.3x7.7, symbol Device:C_Polarized
- added C108: 100µF/16V, Capacitor_SMD:CP_Elec_6.3x5.8, symbol Device:C_Polarized
- BAT101: footprint MyPower:KEYSTONE_1042 -> Battery:BatteryHolder_Keystone_1042_1x18650
- C103, C104, C107: value 100µF/10V -> 100µF/16V; footprint Capacitor_SMD:CP_Elec_6.3x7.7 -> Capacitor_SMD:CP_Elec_6.3x5.8
- D102: value BAV16W -> SL42; footprint Diode_SMD:D_SOD-123 -> Diode_SMD:D_SMC_Handsoldering
- L101, L102: footprint Inductor_SMD:L_6.3x6.3_H3 -> Inductor_SMD:L_12x12mm_H8mm
- R103: value 100K -> 1; footprint Resistor_SMD:R_0805_2012Metric_Pad1.20x1.40mm_HandSolder -> Resistor_SMD:R_1206_3216Metric_Pad1.30x1.75mm_HandSolder
- R104: value 1 -> 1K
- R105: value 1K -> 100K
- T101: value BUK7880-55A -> DMT6009LCT; footprint Package_TO_SOT_SMD:SOT-223-3_TabPin2 -> Package_TO_SOT_THT:TO-220-3_Horizontal_TabDown
Connections:
- net +BATT: now also C108.1
- net Current: now also R104.2; no longer R105.2, TP103.1
- net GND: now also R105.2, C108.2; no longer R104.2
- net Switch: now also R105.1; no longer R103.1
- net Boost: now reaches C103.1, D102.1 (K), L102.1
- net Shunt: now reaches D104.1 (K), R104.1
- net Shunt: now also R103.1, TP103.1; no longer R105.1
- net LED: now reaches D103.1 (K), D104.2 (A)
Other:
- moved on the sheet: C106, D102, D103, L101, L102, TP103, TP105
