File: DiverFlasher/pcb/LED_Flasher.kicad_pcb (KiCad board)
At the start: 2 copper layers, 105 x 24 mm, 30 parts, among them IC101 PIC16LF15313, J101 SKEDD6, SW101 MK15-C2, T101 DMT6009LCT

Commit message: DRC errors removed, finished
Parts:
- T101: footprint Package_TO_SOT_THT:TO-220-3_Horizontal_TabDown -> Package_TO_SOT_THT:TO-220-3_Vertical
- moved R105 17.1 mm to (129.0, 116.4), turned to 180 degrees
- moved C108 7.03 mm to (138.8, 108.0)
- moved C104 6.52 mm to (138.8, 100.2)
- moved T101 4.39 mm to (138.0, 116.2), turned to 0 degrees
- moved R106 3.40 mm to (81.2, 112.8), turned to 180 degrees
- moved TP106 3.25 mm to (70.0, 102.2)
- moved R102 2.90 mm to (73.6, 101.0)
- moved IC101 2.24 mm to (79.7, 106.9)
- moved TP105 2.15 mm to (99.8, 109.8)
- moved TP102 2.10 mm to (132.6, 118.0)
- moved TP104 1.12 mm to (59.9, 113.3)
- moved C107 1.02 mm to (66.5, 115.7)
- moved C102 0.70 mm to (81.2, 115.0)
- moved L102 0.40 mm to (120.5, 107.6)
Routing:
- net /Current: track 56.4 -> 48.7 mm
- net /PWR_MCU: track 49.9 -> 56.7 mm, vias 0 -> 2
- net /LED_PWR: track 35.7 -> 30.3 mm, vias 3 -> 1
- net /ICSPCLK: track 17.2 -> 22.2 mm, vias 0 -> 1
- net /ICSPDAT: track 29.7 -> 32.6 mm
- net /MCLR!: track 14.1 -> 16.7 mm, vias 1 -> 2
- net /Switch: track 80.3 -> 77.8 mm, vias 1 -> 0
- net /SW_OUT: track 62.3 -> 60.2 mm
- net /DEBUG: track 2.50 -> 3.12 mm
