File: DiverFlasher/pcb/LED_Flasher.kicad_pcb (KiCad board)
At the start: 2 copper layers, 105 x 24 mm, 30 parts, among them IC101 PIC16LF15313, J101 SKEDD6, SW101 MK15-C2, T101 DMT6009LCT

Commit message: Production data with JLCPCB plugin generated
Other:
- board text added: "Rev 1.0"
Changed lines of the file:
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@@
 		(tags "test point SMD pad")
 		(property "Reference" "TP103"
-			(at 0 -2.75 0)
+			(at 0.48 1.64 0)
 			(layer "F.SilkS")
 			(effects
 				(font
-					(size 1 1)
+					(size 0.8 0.8)
 					(thickness 0.15)
 				)
@@
 		(tags "resistor handsolder")
 		(property "Reference" "R103"
-			(at -0.8 2 0)
+			(at -0.08 1.73 0)
 			(layer "F.SilkS")
 			(effects
@@
 		(layer "Edge.Cuts")
 	)
+	(gr_text "Rev 1.0"
+		(at 52.18 100.05 0)
+		(layer "F.Cu")
+		(effects
+			(font
+				(size 1.5 1.5)
+				(thickness 0.3)
+				(bold yes)
+			)
+			(justify left bottom)
+		)
+	)
 	(gr_text "Diver flasher"
 		(at 84.5 117 0)
@@
 			(effects
 				(font
+					(size 1 1)
+					(thickness 0.15)
+				)
+			)
+		)
+	)
+	(dimension
+		(type orthogonal)
+		(layer "User.1")
+		(pts
+			(xy 155 120) (xy 155 96)
+		)
+		(height 3.05)
+		(orientation 1)
+		(format
+			(prefix "")
+			(suffix "")
+			(units 3)
+			(units_format 1)
+			(precision 4)
+		)
+		(style
+			(thickness 0.1)
+			(arrow_length 1.27)
+			(text_position_mode 0)
+			(arrow_direction outward)
+			(extension_height 0.58642)
+			(extension_offset 0.5)
+			(keep_text_aligned yes)
+		)
+		(gr_text "24,0000 mm"
+			(at 156.9 108 90)
+			(layer "User.1")
+			(effects
+				(font
+					(size 1 1)
+					(thickness 0.15)
+				)
+			)
+		)
+	)
+	(dimension
+		(type orthogonal)
+		(layer "User.1")
+		(pts
+			(xy 50 96) (xy 155 96)
+		)
+		(height -4)
+		(orientation 0)
+		(format
+			(prefix "")
+			(suffix "")
+			(units 3)
+			(units_format 1)
+			(precision 4)
+		)
+		(style
+			(thickness 0.1)
+			(arrow_length 1.27)
+			(text_position_mode 0)
+			(arrow_direction outward)
+			(extension_height 0.58642)
+			(extension_offset 0.5)
+			(keep_text_aligned yes)
+		)
+		(gr_text "105,0000 mm"
+			(at 102.5 90.85 0)
+			(layer "User.1")
+			(effects
+				(font

Commit message: Side view of the PCB on measurement layer added.
Other:
- board text added: "Batteriehalter mit 18650 Li/Io-Batterie"
- board text added: "Elko"
- board text added: "PCB 1,6mm"
- board text added: "Power Induktivität"
- board text added: "Sensor"
- board text added: "Side View"
Changed lines of the file:
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@@
 		(35 "F.Fab" user)
 		(33 "B.Fab" user)
-		(39 "User.1" user)
+		(39 "User.1" user "Measures.1")
 		(41 "User.2" user)
 		(43 "User.3" user)
@@
 		(layer "Edge.Cuts")
 	)
+	(gr_rect
+		(start 59.4 59.5)
+		(end 79.4 74.5)
+		(stroke
+			(width 0.1)
+			(type default)
+		)
+		(fill no)
+		(layer "User.1")
+	)
+	(gr_circle
+		(center 69.561258 71.1)
+		(end 86.561258 71.1)
+		(stroke
+			(width 0.1)
+			(type dash)
+		)
+		(fill no)
+		(layer "User.1")
+	)
+	(gr_line
+		(start 59.15 76.85)
+		(end 54.9 79.5)
+		(stroke
+			(width 0.1)
+			(type default)
+		)
+		(layer "User.1")
+	)
+	(gr_rect
+		(start 75.6 76.5)
+		(end 81.6 82.5)
+		(stroke
+			(width 0.1)
+			(type default)
+		)
+		(fill no)
+		(layer "User.1")
+	)
+	(gr_rect
+		(start 57.6 74.7)
+		(end 81.6 76.3)
+		(stroke
+			(width 0.1)
+			(type default)
+		)
+		(fill no)
+		(layer "User.1")
+	)
+	(gr_rect
+		(start 63.6 76.5)
+		(end 75.6 86.5)
+		(stroke
+			(width 0.1)
+			(type solid)
+		)
+		(fill no)
+		(layer "User.1")
+	)
+	(gr_rect
+		(start 58.4 76.4)
+		(end 59.9 77.3)
+		(stroke
+			(width 0.1)
+			(type default)
+		)
+		(fill no)
+		(layer "User.1")
+	)
+	(gr_arc
+		(start 59.4 59.5)
+		(mid 69.4 54.5)
+		(end 79.4 59.5)
+		(stroke
+			(width 0.1)
+			(type default)
+		)
+		(layer "User.1")
+	)
 	(gr_text "Rev 1.0"
 		(at 52.18 100.05 0)
@@
 		)
 	)
+	(gr_text "Side View\n"
+		(at 61.9 53.5 0)
+		(layer "User.1")
+		(effects
+			(font
+				(size 2 2)
+				(thickness 0.15)
+			)
+			(justify left bottom)
+		)
+	)
+	(gr_text "Sensor\n"
+		(at 61.7 81.8 90)
+		(layer "User.1")
+		(effects
+			(font
+				(size 1 1)
+				(thickness 0.2)
+				(bold yes)
+			)
+			(justify left bottom)
+		)
+	)
+	(gr_text "PCB 1,6mm"
+		(at 65.2 75.9 0)
+		(layer "User.1")
+		(effects
+			(font
+				(size 1 1)
+				(thickness 0.15)
+			)
+			(justify left bottom)
+		)
+	)
+	(gr_text "Elko\n"
+		(at 77 79.5 0)
+		(layer "User.1")
+		(effects
+			(font
+				(size 1 1)
+				(thickness 0.15)
+			)
+			(justify left bottom)
+		)
+	)
+	(gr_text "Power\nInduktivität\n"
+		(at 66 82.9 0)
+		(layer "User.1")
+		(effects
+			(font
+				(size 1 1)
+				(thickness 0.15)
+			)
+			(justify left bottom)
+		)
+	)
+	(gr_text "Batteriehalter mit \n18650 Li/Io-Batterie "
+		(at 61.8 64.3 0)
+		(layer "User.1")
+		(effects
+			(font
+				(size 1 1)
+				(thickness 0.15)
+			)
+			(justify left bottom)
+		)
+	)
+	(dimension
+		(type aligned)
+		(layer "User.1")
+		(pts
+			(xy 54.8 79.6) (xy 59.15 76.85)
+		)
+		(height -5.941513)
+		(format
+			(prefix "")
+			(suffix "")
+			(units 3)
+			(units_format 1)
+			(precision 4)
+		)
+		(style
+			(thickness 0.1)
+			(arrow_length 1.27)
+			(text_position_mode 0)
+			(arrow_direction outward)
+			(extension_height 0.58642)
+			(extension_offset 0.5)
+			(keep_text_aligned yes)
+		)
+		(gr_text "5,1464 mm"
+			(at 53.18559 72.230842 32.30041551)
+			(layer "User.1")
+			(effects
+				(font
+					(size 1 1)
+					(thickness 0.15)
+				)
+			)
+		)
+	)
 	(dimension
 		(type orthogonal)
@@
 			(layer "User.1")
 			(effects
+				(font
+					(size 1 1)
+					(thickness 0.15)
+				)
+			)
+		)
+	)
+	(dimension
+		(type orthogonal)
+		(layer "User.1")
+		(pts
+			(xy 69.561258 88.1) (xy 69.561258 54.1)
+		)
+		(height 19.338742)
+		(orientation 1)
+		(format
+			(prefix "")
+			(suffix "")
+			(units 3)
+			(units_format 1)
+			(precision 4)
+		)
+		(style
+			(thickness 0.1)
+			(arrow_length 1.27)
+			(text_position_mode 0)
+			(arrow_direction outward)
+			(extension_height 0.58642)
+			(extension_offset 0.5)
+			(keep_text_aligned yes)
+		)
+		(gr_text "34,0000 mm"
+			(at 87.75 71.1 90)
+			(layer "User.1")
+			(effects

Commit message: Platineneigenschaften und Lagenaufbau au PCB-Sheet hinzugefügt.
Other:
- board text added: "0"
- board text added: "0 mm"
- board text added: "0,0000 mm / 0,0000 mm"
- board text added: "0,01 mm"
- board text added: "0,02"
- board text added: "0,035 mm"
- board text added: "0,3000 mm"
- board text added: "1"
- board text added: "1,51 mm"
- board text added: "1,6000 mm"
- board text added: "105,0000 mm x 24,0000 mm"
- board text added: "2"
- board text added: "3,3"
- board text added: "4,5"
- board text added: "Abmessungen der Platine:"
- board text added: "B.Cu"
- board text added: "B.Mask"
- board text added: "B.Paste"
- board text added: "B.Silkscreen"
- board text added: "Bottom Silk Screen"
- board text added: "Bottom Solder Mask"
- board text added: "Bottom Solder Paste"
- board text added: "Castellated Pads:"
- board text added: "Dicke (mm)"
- board text added: "Dielektrikum"
- board text added: "Epsilon R"
- board text added: "F.Cu"
- board text added: "F.Mask"
- board text added: "F.Paste"
- board text added: "F.Silkscreen"
- board text added: "FR4"
- board text added: "Farbe"
- board text added: "HAL lead-free"
- board text added: "Impedanzkontrolle:"
- board text added: "Kupferlagenanzahl:"
- board text added: "Kupferoberfläche:"
- board text added: "Lagenname"
- board text added: "Material"
- board text added: "Metallisierte Platinenkante:"
- board text added: "Min Leiterbahn/abstand:"
- board text added: "Min Lochdurchmesser:"
- board text added: "Nein"
- board text added: "Not specified"
- board text added: "PLATINEN-EIGENSCHAFTEN"
- board text added: "Platinen-Dicke:"
- board text added: "Randsteckverbinder:"
- board text added: "Tangens des Verlustwinkels"
- board text added: "Top Silk Screen"
- board text added: "Top Solder Mask"
- board text added: "Top Solder Paste"
- board text added: "Typ"
- board text added: "copper"
- board text added: "core"
