File: DiverFlasher/pcb/LED_Flasher.kicad_sch (KiCad schematic)
At the start: 30 parts, among them IC101 PIC16LF15313, J101 SKEDD6, SW101 MK15-C2, T101 DMT6009LCT

Commit message: DRC errors removed, finished
Parts:
- T101: footprint Package_TO_SOT_THT:TO-220-3_Horizontal_TabDown -> Package_TO_SOT_THT:TO-220-3_Vertical
Changed lines of the file:
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@@
 			)
 		)
-		(property "Footprint" "Package_TO_SOT_THT:TO-220-3_Horizontal_TabDown"
+		(property "Footprint" "Package_TO_SOT_THT:TO-220-3_Vertical"
 			(at 106.68 62.865 0)
 			(effects

Commit message: Ruhestrom hinzugefügt (50µA)
Other:
- note added: "IRuhe ca. 50µA"
Changed lines of the file:
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@@
 		(comment 1 "Dipl.-Ing. Jürgen Eggeling")
+	)
+	(text "IRuhe ca. 50µA"
+		(exclude_from_sim no)
+		(at 59.182 109.22 0)
+		(effects
+			(font
+				(size 1.27 1.27)
+			)
+		)
 	)
 	(text_box "Version overview\nV1.0 integrated booster circuit (too weak)\nV1.1 home brew booster circuit"
