File: DiverMarker/pcb/LED_Marker.kicad_pcb (KiCad board)
At the start: 2 copper layers, 75 x 20 mm, 26 parts, among them IC101 PIC16LF15313, J101 SKEDD6, Q100 BST-52, Q101 BST-52, SW101 MK15-C2

Commit message: Side View on Measurment layer added
Other:
- board text added: "Batteriehalter mit AA-Batterie"
- board text added: "Elko"
- board text added: "PCB"
- board text added: "Sensor"
- board text added: "Side View"
Changed lines of the file:
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@@
 		(35 "F.Fab" user)
 		(33 "B.Fab" user)
-		(39 "User.1" user)
+		(39 "User.1" user "Measurement")
 		(41 "User.2" user)
 		(43 "User.3" user)
@@
 		(layer "Edge.Cuts")
 	)
+	(gr_rect
+		(start 110.8 80.468454)
+		(end 112.3 81.368454)
+		(stroke
+			(width 0.1)
+			(type default)
+		)
+		(fill no)
+		(layer "User.1")
+	)
+	(gr_line
+		(start 120 86.268454)
+		(end 120 60.268454)
+		(stroke
+			(width 0.05)
+			(type dash_dot)
+		)
+		(layer "User.1")
+	)
+	(gr_rect
+		(start 110 78.668454)
+		(end 130 80.268454)
+		(stroke
+			(width 0.2)
+			(type solid)
+		)
+		(fill no)
+		(layer "User.1")
+	)
+	(gr_rect
+		(start 111.5 62.768454)
+		(end 128.5 78.268454)
+		(stroke
+			(width 0.1)
+			(type default)
+		)
+		(fill no)
+		(layer "User.1")
+	)
+	(gr_rect
+		(start 119.6 80.468454)
+		(end 127.6 88.468454)
+		(stroke
+			(width 0.1)
+			(type default)
+		)
+		(fill no)
+		(layer "User.1")
+	)
+	(gr_circle
+		(center 120 75.5)
+		(end 135.5 75.5)
+		(stroke
+			(width 0.1)
+			(type dash)
+		)
+		(fill no)
+		(layer "User.1")
+	)
 	(gr_line
 		(start 98.27 110)
@@
 		)
 	)
+	(gr_text "PCB"
+		(at 118.8 79.968454 0)
+		(layer "User.1")
+		(effects
+			(font
+				(size 0.8 0.8)
+				(thickness 0.2)
+				(bold yes)
+			)
+			(justify left bottom)
+		)
+	)
+	(gr_text "Batteriehalter\nmit AA-Batterie"
+		(at 114 70.268454 0)
+		(layer "User.1")
+		(effects
+			(font
+				(size 1 1)
+				(thickness 0.15)
+			)
+			(justify left bottom)
+		)
+	)
+	(gr_text "Elko"
+		(at 121.9 83.068454 0)
+		(layer "User.1")
+		(effects
+			(font
+				(size 1 1)
+				(thickness 0.15)
+			)
+			(justify left bottom)
+		)
+	)
+	(gr_text "Sensor\n"
+		(at 113.5 81.668454 0)
+		(layer "User.1")
+		(effects
+			(font
+				(size 1 1)
+				(thickness 0.2)
+				(bold yes)
+			)
+			(justify left bottom)
+		)
+	)
+	(gr_text "Side View"
+		(at 113.1 59.4 0)
+		(layer "User.1")
+		(effects
+			(font
+				(size 2 2)
+				(thickness 0.15)
+			)
+			(justify left bottom)
+		)
+	)
 	(dimension
 		(type orthogonal)
@@
 			(layer "User.1")
 			(effects
+				(font
+					(size 1 1)
+					(thickness 0.15)
+				)
+			)
+		)
+	)
+	(dimension
+		(type orthogonal)
+		(layer "User.1")
+		(pts
+			(xy 120 60) (xy 120 91)
+		)
+		(height 20)
+		(orientation 1)
+		(format
+			(prefix "")
+			(suffix "")
+			(units 3)
+			(units_format 1)
+			(precision 4)
+		)
+		(style
+			(thickness 0.1)
+			(arrow_length 1.27)
+			(text_position_mode 0)
+			(arrow_direction outward)
+			(extension_height 0.58642)
+			(extension_offset 0.5)
+			(keep_text_aligned yes)
+		)
+		(gr_text "31,0000 mm"
+			(at 138.85 75.5 90)
+			(layer "User.1")
+			(effects

Commit message: PCB informations added
Other:
- board text added: "0"
- board text added: "0 mm"
- board text added: "0,0000 mm / 0,0000 mm"
- board text added: "0,01 mm"
- board text added: "0,02"
- board text added: "0,035 mm"
- board text added: "0,3000 mm"
- board text added: "1"
- board text added: "1,51 mm"
- board text added: "1,6000 mm"
- board text added: "2"
- board text added: "3,3"
- board text added: "4,5"
- board text added: "75,0000 mm x 20,0000 mm"
- board text added: "Abmessungen der Platine:"
- board text added: "B.Cu"
- board text added: "B.Mask"
- board text added: "B.Paste"
- board text added: "B.Silkscreen"
- board text added: "Bottom Silk Screen"
- board text added: "Bottom Solder Mask"
- board text added: "Bottom Solder Paste"
- board text added: "Castellated Pads:"
- board text added: "Dicke (mm)"
- board text added: "Dielektrikum 1"
- board text added: "Epsilon R"
- board text added: "F.Cu"
- board text added: "F.Mask"
- board text added: "F.Paste"
- board text added: "F.Silkscreen"
- board text added: "FR4"
- board text added: "Farbe"
- board text added: "HAL lead-free"
- board text added: "Impedanzkontrolle:"
- board text added: "Kupferlagenanzahl:"
- board text added: "Kupferoberfläche:"
- board text added: "Lagenname"
- board text added: "Material"
- board text added: "Metallisierte Platinenkante:"
- board text added: "Min Leiterbahn/abstand:"
- board text added: "Min Lochdurchmesser:"
- board text added: "Nein"
- board text added: "Not specified"
- board text added: "PLATINEN-EIGENSCHAFTEN"
- board text added: "Platinen-Dicke:"
- board text added: "Randsteckverbinder:"
- board text added: "Red"
- board text added: "Tangens des Verlustwinkels"
- board text added: "Top Silk Screen"
- board text added: "Top Solder Mask"
- board text added: "Top Solder Paste"
- board text added: "Typ"
- board text added: "White"
- board text added: "copper"
- board text added: "core"
